Commit message: Imported upstream version '1.9.4' of 'upstream'

File: test/robots/pr2/shoulder_v0/shoulder.urdf.xacro (robot description, xacro)
@@ -10,6 +10,6 @@
   <xacro:include filename="$(find xacro)/test/robots/pr2/shoulder_v0/shoulder.transmission.xacro" />
   <xacro:include filename="$(find xacro)/test/robots/pr2/common.xacro" />
-  <xacro:property name="shoulder_lift_length" value="0.10" />  <!--TODO Define and give source-->
-  <xacro:property name="shoulder_lift_radius" value="0.12" />  <!--TODO Define and give source-->
+  <property name="shoulder_lift_length" value="0.10" />  <!--TODO Define and give source-->
+  <property name="shoulder_lift_radius" value="0.12" />  <!--TODO Define and give source-->
  <!-- ============================   Shoulder   ============================ -->
   <xacro:macro name="pr2_shoulder_v0" params="side parent reflect *origin">
@@ -17,5 +17,5 @@
     <joint name="${side}_shoulder_pan_joint" type="revolute">
       <axis xyz="0 0 1" />
-      <xacro:insert_block name="origin" /> <!-- transform from parent link to this joint frame -->
+      <insert_block name="origin" /> <!-- transform from parent link to this joint frame -->
       <parent link="${parent}"/>
       <child link="${side}_shoulder_pan_link"/>
@@ -99,5 +99,5 @@
     <joint name="${side}_upper_arm_roll_joint" type="revolute">
       <axis xyz="1 0 0" />
-      <xacro:insert_block name="origin" />
+      <insert_block name="origin" />
       <parent link="${parent}" />
       <child link="${side}_upper_arm_roll_link"/>

File: test/robots/pr2/tilting_laser_v0/tilting_laser.urdf.xacro (robot description, xacro)
@@ -14,5 +14,5 @@
       <calibration falling="${laser_calib_ref}" />
       <dynamics damping="0.008" />
-      <xacro:insert_block name="origin" />
+      <insert_block name="origin" />
       <parent link="${parent}"/>
       <child link="${name}_mount_link"/>
