Commit message: Imported upstream version '2.0.8' of 'upstream'

File: test/include2.xacro (robot description, xacro)
@@ -1,4 +1,7 @@
 <a xmlns:xacro="http://www.ros.org/wiki/xacro">
 	<xacro:property name="var" value="2"/>
+	<xacro:property name="inner" value="int"/>
+	<xacro:property name="arg" value="default"/>
 	<xacro:macro name="foo"><inc2/></xacro:macro>
+	<xacro:macro name="bar" params="arg"><a arg="${arg}" var="${var}" ext="${ext}"/></xacro:macro>
 </a>

File: test/robots/pr2/gripper_v0/gripper.gazebo.xacro (robot description, xacro)
@@ -22,5 +22,4 @@
       <kp value="1000000.0" />
       <kd value="1.0" />
-      <!-- for "${prefix}_l_finger_joint"-->
     </gazebo>
     <gazebo reference="${prefix}_l_finger_joint">

File: test/robots/pr2/sensors/kinect_prosilica_camera.urdf.xacro (robot description, xacro)
@@ -40,8 +40,4 @@
       </collision>
     </link>
-    <!-- plugin for updating structure pose \
-    <xacro:kinect_prosilica_gazebo joint_name="${name}_kinect_prosilica_joint"
-                                   link_name="${name}_kinect_prosilica_link" />
-    -->
     <!-- kinect ir sensor physical attachment -->
     <joint name="${name}_kinect_ir_joint" type="fixed">
